File: rasbperryPiRobotSchield/rasbperryPI.brd (EAGLE design)
At the start: 60.6 x 54.6 mm, 22 parts, among them X1 SSW-104-02-S-D

Commit message: next
Parts:
- removed JP15, JP16: (no value), jumper:JP1
- added A_MOTOR, B_MOTOR: (no value), jumper:JP1
- moved POWER_RPI 32.1 mm to (64.8, 69.2), turned to 180 degrees
- moved PWM_IN 4.26 mm to (72.4, 62.9)
- moved +5V 4.02 mm to (72.4, 69.2), turned to 180 degrees
- moved +12V 3.81 mm to (72.4, 74.9), turned to 0 degrees
- moved TB1 2.54 mm to (50.8, 68.8)
Connections:
- net N$1 renamed SDA
- net N$2 renamed SCL
- net GND: now also U$1.25
- net N$17: now also B_MOTOR.1; no longer JP15.1
- net N$18: now also B_MOTOR.2; no longer JP15.2
- net N$19: now also A_MOTOR.1; no longer JP16.1
- net N$20: now also A_MOTOR.2; no longer JP16.2
Routing:
- net 5V0@1: track 12.0 -> 45.6 mm
- net GND: track 187.9 -> 207.6 mm
- net N$12: track 29.8 -> 44.3 mm
- net +5V: track 142.6 -> 128.9 mm
- net N$15: track 29.8 -> 36.3 mm
- net N$16: track 25.2 -> 31.7 mm
- net N$11: track 12.0 -> 15.9 mm
- net VCC: track 11.5 -> 15.3 mm
- net N$26: track 3.81 -> 6.35 mm
- net N$25: track 3.81 -> 6.35 mm
- net N$24: track 3.81 -> 6.35 mm
- net N$23: track 3.81 -> 6.35 mm
- net N$17: track 17.6 -> 16.2 mm

Commit message: next rasbperry pi shield
Parts:
- added +7V, +7V1: (no value), jumper:JP1
- added JP1: (no value), jumper:JP2
- added PWM1: PWMPCB, PWM_I2C:PWM
- U$1: device RPI-Zero:RASPBERRYPI_BASTELSTUBE_V13_RASPI_BOARD_B+_FULL -> RPI-Zero:RASP_PI_ZERO_BOARD_FULL
- moved POWER_RPI 53.2 mm to (15.9, 90.2), turned to 90 degrees
- moved JP4 44.0 mm to (72.4, 59.1), flipped to the top
- moved U$1 40.5 mm to (16.5, 27.0)
- moved A_MOTOR 30.7 mm to (48.4, 88.9), turned to 270 degrees
- moved +5V 26.1 mm to (55.2, 88.9), turned to 90 degrees
- moved PWM_IN 26.0 mm to (73.0, 88.9), turned to 270 degrees
- moved B_MOTOR 22.6 mm to (42.7, 88.9), turned to 270 degrees
- moved +12V 17.3 mm to (62.2, 88.9), turned to 270 degrees
- moved I2C 1.80 mm to (38.1, 31.8)
- moved SERIAL 1.80 mm to (27.9, 31.8)
- moved JP10 1.27 mm to (73.7, 31.8)
- moved JP2 1.27 mm to (29.2, 34.9)
- moved JP3 1.27 mm to (29.2, 44.5)
- moved JP7 1.27 mm to (63.5, 31.8)
- moved JP5 1.27 mm to (36.8, 44.5)
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Connections:
- new net N$1: +7V.2, +7V1.2, PWM1.V+$1
- new net N$2: JP4.1, U$1.36
- new net N$31: JP4.2, U$1.38
- new net N$34: JP4.3, U$1.40
- net +5V: now also JP1.3, PWM1.VCC$1; no longer JP4.3
- net A_SCL: now also JP1.1, PWM1.SCL$1; no longer JP4.1
- net A_SDA: now also JP1.2, PWM1.SDA$1; no longer JP4.2
- net GND: now also +7V.1, PWM1.GND$1, U$1.30, U$1.34, U$1.39
- net VCC: now also +7V1.1
Routing:
- net GND: track 207.6 -> 374.9 mm
- net +5V: track 128.9 -> 213.6 mm, vias 0 -> 2
- net A_SDA: track 4.44 -> 61.3 mm
- net A_SCL: track 4.44 -> 60.0 mm
- net VCC: track 15.3 -> 54.7 mm, vias 0 -> 2
- net N$1: track 0.00 -> 33.6 mm
- net N$11: track 15.9 -> 37.7 mm
- net N$20: track 27.3 -> 12.5 mm
- net N$16: track 31.7 -> 45.7 mm
- net N$15: track 36.3 -> 48.2 mm
- net N$19: track 23.7 -> 12.5 mm
- net N$12: track 44.3 -> 55.0 mm
- net N$18: track 19.9 -> 12.8 mm
- net N$34: track 0.00 -> 4.20 mm
- net N$31: track 0.00 -> 4.20 mm
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Other:
- board size 60.6 x 54.6 mm -> 78.4 x 73.6 mm
- board text added: "GND"
- board text added: "MOTOR OUT"
- board text added: "MTR PWM"
- board text added: "MTR Vcc"
- board text added: "MTR=SRV"
- board text added: "Rpi ON"
- board text added: "Rpi Shileld v2.0"
- board text added: "SRV Vcc"
- board text removed: "Rpi Shileld v1.0"
