File: rasbperryPiRobotSchield/rasbperryPI.brd (EAGLE design)
At the start: 78.4 x 73.6 mm, 26 parts, among them X1 SSW-104-02-S-D

Commit message: next brd
Parts:
- moved I2C 3.81 mm to (38.1, 27.9)
- moved JP10 3.81 mm to (73.7, 27.9)
- moved JP7 3.81 mm to (63.5, 27.9)
- moved SERIAL 3.81 mm to (27.9, 27.9)
Connections:
- net N$15 renamed RX
- net N$16 renamed TX
Routing:
- net +5V: track 213.6 -> 207.2 mm, vias 2 -> 4
- net GND: track 374.9 -> 379.1 mm
- net A_SCL: track 60.0 -> 63.8 mm
- net N$30: track 3.17 -> 6.98 mm
- net N$29: track 3.17 -> 6.98 mm
- net N$28: track 3.17 -> 6.98 mm
- net N$27: track 3.17 -> 6.98 mm
- net N$22: track 3.17 -> 6.98 mm
- net N$21: track 3.17 -> 6.98 mm
- net A_SDA: track 61.3 -> 65.1 mm
- net N$12: track 55.0 -> 56.5 mm
- net N$11: track 37.7 -> 39.2 mm
Other:
- board text added: "RX"
- board text added: "SCL"
- board text added: "SDA"
- board text added: "TX"
