File: rasbperryPiRobotSchield/rasbperryPI.sch (EAGLE design)
At the start: 22 parts, among them X1 SSW-104-02-S-D

Commit message: next
Parts:
- renumbered JP15 to B_MOTOR, JP16 to A_MOTOR
Connections:
- net N$1 renamed SDA
- net N$2 renamed SCL
- net GND: now also U$1.GND@2
Other:
- moved on the sheet: JP5
Changed lines of the file:
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@@
 <grid distance="0.1" unitdist="inch" unit="inch" style="lines" multiple="1" display="no" altdistance="0.01" altunitdist="inch" altunit="inch"/>
 <layers>
-<layer number="1" name="Top" color="4" fill="1" visible="yes" active="no"/>
-<layer number="16" name="Bottom" color="1" fill="1" visible="yes" active="no"/>
-<layer number="17" name="Pads" color="2" fill="1" visible="yes" active="no"/>
-<layer number="18" name="Vias" color="2" fill="1" visible="yes" active="no"/>
-<layer number="19" name="Unrouted" color="6" fill="1" visible="yes" active="no"/>
-<layer number="20" name="Dimension" color="24" fill="1" visible="yes" active="no"/>
-<layer number="21" name="tPlace" color="7" fill="1" visible="yes" active="no"/>
-<layer number="22" name="bPlace" color="7" fill="1" visible="yes" active="no"/>
-<layer number="23" name="tOrigins" color="15" fill="1" visible="yes" active="no"/>
-<layer number="24" name="bOrigins" color="15" fill="1" visible="yes" active="no"/>
-<layer number="25" name="tNames" color="7" fill="1" visible="yes" active="no"/>
-<layer number="26" name="bNames" color="7" fill="1" visible="yes" active="no"/>
-<layer number="27" name="tValues" color="7" fill="1" visible="yes" active="no"/>
-<layer number="28" name="bValues" color="7" fill="1" visible="yes" active="no"/>
+<layer number="1" name="Top" color="4" fill="1" visible="no" active="no"/>
+<layer number="16" name="Bottom" color="1" fill="1" visible="no" active="no"/>
+<layer number="17" name="Pads" color="2" fill="1" visible="no" active="no"/>
+<layer number="18" name="Vias" color="2" fill="1" visible="no" active="no"/>
+<layer number="19" name="Unrouted" color="6" fill="1" visible="no" active="no"/>
+<layer number="20" name="Dimension" color="24" fill="1" visible="no" active="no"/>
+<layer number="21" name="tPlace" color="7" fill="1" visible="no" active="no"/>
+<layer number="22" name="bPlace" color="7" fill="1" visible="no" active="no"/>
+<layer number="23" name="tOrigins" color="15" fill="1" visible="no" active="no"/>
+<layer number="24" name="bOrigins" color="15" fill="1" visible="no" active="no"/>
+<layer number="25" name="tNames" color="7" fill="1" visible="no" active="no"/>
+<layer number="26" name="bNames" color="7" fill="1" visible="no" active="no"/>
+<layer number="27" name="tValues" color="7" fill="1" visible="no" active="no"/>
+<layer number="28" name="bValues" color="7" fill="1" visible="no" active="no"/>
 <layer number="29" name="tStop" color="7" fill="3" visible="no" active="no"/>
 <layer number="30" name="bStop" color="7" fill="6" visible="no" active="no"/>
@@
 <layer number="35" name="tGlue" color="7" fill="4" visible="no" active="no"/>
 <layer number="36" name="bGlue" color="7" fill="5" visible="no" active="no"/>
-<layer number="37" name="tTest" color="7" fill="1" visible="yes" active="no"/>
-<layer number="38" name="bTest" color="7" fill="1" visible="yes" active="no"/>
+<layer number="37" name="tTest" color="7" fill="1" visible="no" active="no"/>
+<layer number="38" name="bTest" color="7" fill="1" visible="no" active="no"/>
 <layer number="39" name="tKeepout" color="4" fill="11" visible="no" active="no"/>
 <layer number="40" name="bKeepout" color="1" fill="11" visible="no" active="no"/>
@@
 <layer number="44" name="Drills" color="7" fill="1" visible="no" active="no"/>
 <layer number="45" name="Holes" color="7" fill="1" visible="no" active="no"/>
-<layer number="46" name="Milling" color="3" fill="1" visible="yes" active="no"/>
-<layer number="47" name="Measures" color="7" fill="1" visible="yes" active="no"/>
-<layer number="48" name="Document" color="7" fill="1" visible="yes" active="no"/>
-<layer number="49" name="Reference" color="7" fill="1" visible="yes" active="no"/>
-<layer number="50" name="dxf" color="7" fill="1" visible="yes" active="no"/>
-<layer number="51" name="tDocu" color="7" fill="1" visible="yes" active="no"/>
-<layer number="52" name="bDocu" color="7" fill="1" visible="yes" active="no"/>
-<layer number="53" name="tGND_GNDA" color="7" fill="1" visible="yes" active="no"/>
-<layer number="54" name="bGND_GNDA" color="7" fill="1" visible="yes" active="no"/>
-<layer number="56" name="wert" color="7" fill="1" visible="yes" active="no"/>
-<layer number="57" name="tCAD" color="7" fill="1" visible="yes" active="no"/>
-<layer number="59" name="tCarbon" color="7" fill="1" visible="yes" active="no"/>
-<layer number="60" name="bCarbon" color="7" fill="1" visible="yes" active="no"/>
+<layer number="46" name="Milling" color="3" fill="1" visible="no" active="no"/>
+<layer number="47" name="Measures" color="7" fill="1" visible="no" active="no"/>
+<layer number="48" name="Document" color="7" fill="1" visible="no" active="no"/>
+<layer number="49" name="Reference" color="7" fill="1" visible="no" active="no"/>
+<layer number="50" name="dxf" color="7" fill="1" visible="no" active="no"/>
+<layer number="51" name="tDocu" color="7" fill="1" visible="no" active="no"/>
+<layer number="52" name="bDocu" color="7" fill="1" visible="no" active="no"/>
+<layer number="53" name="tGND_GNDA" color="7" fill="1" visible="no" active="no"/>
+<layer number="54" name="bGND_GNDA" color="7" fill="1" visible="no" active="no"/>
+<layer number="56" name="wert" color="7" fill="1" visible="no" active="no"/>
+<layer number="57" name="tCAD" color="7" fill="1" visible="no" active="no"/>
+<layer number="59" name="tCarbon" color="7" fill="1" visible="no" active="no"/>
+<layer number="60" name="bCarbon" color="7" fill="1" visible="no" active="no"/>
 <layer number="90" name="Modules" color="5" fill="1" visible="yes" active="yes"/>
 <layer number="91" name="Nets" color="2" fill="1" visible="yes" active="yes"/>
@@
 <part name="P+5" library="supply1" deviceset="+5V" device=""/>
 <part name="P+6" library="supply1" deviceset="+5V" device=""/>
-<part name="JP15" library="jumper" deviceset="JP1E" device=""/>
-<part name="JP16" library="jumper" deviceset="JP1E" device=""/>
+<part name="B_MOTOR" library="jumper" deviceset="JP1E" device=""/>
+<part name="A_MOTOR" library="jumper" deviceset="JP1E" device=""/>
 <part name="SERIAL" library="jumper" deviceset="JP1E" device=""/>
 <part name="SUPPLY1" library="supply2" deviceset="VCC" device=""/>
@@
 <instance part="JP3" gate="1" x="27.94" y="104.14"/>
 <instance part="JP4" gate="1" x="33.02" y="-22.86"/>
-<instance part="JP5" gate="1" x="30.48" y="33.02" rot="R180"/>
+<instance part="JP5" gate="1" x="27.94" y="17.78" rot="R180"/>
 <instance part="GND4" gate="1" x="22.86" y="-27.94"/>
 <instance part="GND5" gate="1" x="15.24" y="91.44"/>
 <instance part="P+2" gate="1" x="35.56" y="-27.94" rot="R180"/>
-<instance part="+3V2" gate="G$1" x="33.02" y="40.64"/>
+<instance part="+3V2" gate="G$1" x="33.02" y="25.4"/>
 <instance part="+3V3" gate="G$1" x="-15.24" y="55.88" rot="R270"/>
 <instance part="I2C" gate="A" x="33.02" y="-40.64" rot="R180"/>
-<instance part="GND6" gate="1" x="83.82" y="17.78"/>
+<instance part="GND6" gate="1" x="63.5" y="33.02"/>
 <instance part="JP8" gate="1" x="116.84" y="-10.16"/>
 <instance part="JP9" gate="1" x="129.54" y="-10.16"/>
@@
 <instance part="P+5" gate="1" x="91.44" y="106.68" rot="R180"/>
 <instance part="P+6" gate="1" x="101.6" y="142.24"/>
-<instance part="JP15" gate="A" x="76.2" y="149.86"/>
-<instance part="JP16" gate="A" x="86.36" y="149.86"/>
+<instance part="B_MOTOR" gate="A" x="76.2" y="149.86"/>
+<instance part="A_MOTOR" gate="A" x="86.36" y="149.86"/>
 <instance part="SERIAL" gate="A" x="20.32" y="-40.64" rot="R180"/>
 <instance part="SUPPLY1" gate="G$1" x="147.32" y="76.2" rot="R90"/>
@@
 <pinref part="GND11" gate="1" pin="GND"/>
 </segment>
+<segment>
+<pinref part="U$1" gate="G$1" pin="GND@2"/>
+<pinref part="GND6" gate="1" pin="GND"/>
+<wire x1="63.5" y1="35.56" x2="55.88" y2="45.72" width="0.1524" layer="91"/>
+</segment>
 </net>
 <net name="+5V" class="0">
@@
 <pinref part="JP5" gate="1" pin="1"/>
 <pinref part="+3V2" gate="G$1" pin="+3V3"/>
-<wire x1="33.02" y1="35.56" x2="33.02" y2="38.1" width="0.1524" layer="91"/>
+<wire x1="30.48" y1="20.32" x2="33.02" y2="22.86" width="0.1524" layer="91"/>
 </segment>
 <segment>
@@
 <segment>
 <pinref part="TB1" gate="G$1" pin="B1"/>
-<pinref part="JP15" gate="A" pin="1"/>
+<pinref part="B_MOTOR" gate="A" pin="1"/>
 <wire x1="76.2" y1="139.7" x2="76.2" y2="147.32" width="0.1524" layer="91"/>
 </segment>
@@
 <segment>
 <pinref part="TB1" gate="G$1" pin="B2"/>
-<pinref part="JP15" gate="A" pin="2"/>
+<pinref part="B_MOTOR" gate="A" pin="2"/>
 <wire x1="81.28" y1="139.7" x2="78.74" y2="147.32" width="0.1524" layer="91"/>
 </segment>
@@
 <segment>
 <pinref part="TB1" gate="G$1" pin="A2"/>
-<pinref part="JP16" gate="A" pin="1"/>
+<pinref part="A_MOTOR" gate="A" pin="1"/>
 <wire x1="86.36" y1="139.7" x2="86.36" y2="147.32" width="0.1524" layer="91"/>
 </segment>
@@
 <segment>
 <pinref part="TB1" gate="G$1" pin="A1"/>
-<pinref part="JP16" gate="A" pin="2"/>
+<pinref part="A_MOTOR" gate="A" pin="2"/>
 <wire x1="91.44" y1="139.7" x2="88.9" y2="147.32" width="0.1524" layer="91"/>
 </segment>
@@
 </segment>
 </net>
-<net name="N$1" class="0">
+<net name="SDA" class="0">
 <segment>
 <pinref part="U$1" gate="G$1" pin="GPIO2/SDA1"/>
 <pinref part="JP5" gate="1" pin="2"/>
-<wire x1="27.94" y1="45.72" x2="30.48" y2="35.56" width="0.1524" layer="91"/>
-</segment>
-</net>
-<net name="N$2" class="0">
+<wire x1="27.94" y1="45.72" x2="27.94" y2="20.32" width="0.1524" layer="91"/>
+<label x="30.48" y="27.94" size="1.778" layer="95" xref="yes"/>
+</segment>
+</net>
+<net name="SCL" class="0">
 <segment>
 <pinref part="U$1" gate="G$1" pin="GPIO3/SCL1"/>
 <pinref part="JP5" gate="1" pin="3"/>
-<wire x1="30.48" y1="45.72" x2="27.94" y2="35.56" width="0.1524" layer="91"/>
-</segment>
-</net>
+<wire x1="30.48" y1="45.72" x2="25.4" y2="20.32" width="0.1524" layer="91"/>
+<label x="20.32" y="20.32" size="1.778" layer="95" rot="R180" xref="yes"/>
+</segment>
+</net>

Commit message: next rasbperry pi shield
Parts:
- added +7V, +7V1: (no value), jumper:JP1E
- added JP1: (no value), jumper:JP2E
- added PWM1: PWMPCB, PWM_I2C:PWMPCB
Connections:
- new net N$1: +7V.2, +7V1.2, PWM1.V+_1
- new net N$2: JP4.1, U$1.GPIO16
- new net N$31: JP4.2, U$1.GPIO20
- new net N$34: JP4.3, U$1.GPIO21
- net +5V: now also JP1.3, PWM1.VCC_1; no longer JP4.3
- net A_SCL: now also JP1.1, PWM1.SCL_1; no longer JP4.1
- net A_SDA: now also JP1.2, PWM1.SDA_1; no longer JP4.2
- net GND: now also +7V.1, PWM1.GND_1, U$1.GND@3, U$1.GND@6, U$1.GND@7
- net VCC: now also +7V1.1
Other:
- moved on the sheet: JP4, U$1

Commit message: next brd
Connections:
- net N$15 renamed RX
- net N$16 renamed TX
Changed lines of the file:
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@@
 </segment>
 </net>
-<net name="N$15" class="0">
+<net name="RX" class="0">
 <segment>
 <pinref part="JP3" gate="1" pin="3"/>
 <pinref part="U$1" gate="G$1" pin="RXD0/GPIO15"/>
 <wire x1="30.48" y1="101.6" x2="30.48" y2="91.44" width="0.1524" layer="91"/>
+<label x="33.02" y="96.52" size="1.778" layer="95" xref="yes"/>
 </segment>
 </net>
-<net name="N$16" class="0">
+<net name="TX" class="0">
 <segment>
 <pinref part="JP3" gate="1" pin="2"/>
 <pinref part="U$1" gate="G$1" pin="TXD0/GPIO14"/>
 <wire x1="27.94" y1="101.6" x2="27.94" y2="91.44" width="0.1524" layer="91"/>
+<label x="25.4" y="96.52" size="1.778" layer="95" rot="R180" xref="yes"/>
 </segment>
 </net>
